File: kicad/attiny13a/attiny13a.sch (KiCad schematic (older format))
At the start: 5 parts, among them P1 CONN_01X04, P2 CONN_01X04, P3 CONN_01X06, U1 ATTINY13A-SSU

Commit message: Add atiny13 full schematic/pcb
Parts:
- C1: footprint (none) -> Capacitors_SMD:C_0805_HandSoldering
- P1, P2: footprint (none) -> Socket_Strips:Socket_Strip_Straight_1x04
- P3: footprint (none) -> Socket_Strips:Socket_Strip_Straight_1x06
- U1: footprint SO8 -> Housings_SOIC:SOIC-8_3.9x4.9mm_Pitch1.27mm
Changed lines of the file:
@@
 F 0 "U1" H 5300 3717 50  0000 C CNN
 F 1 "ATTINY13A-SSU" H 5300 3626 50  0000 C CNN
-F 2 "SO8" H 5900 3200 50  0001 C CIN
+F 2 "Housings_SOIC:SOIC-8_3.9x4.9mm_Pitch1.27mm" H 5900 3200 50  0001 C CIN
 F 3 "" H 4500 3550 50  0001 C CNN
 	1    5300 3200
@@
 F 0 "P1" V 4890 2062 50  0000 R CNN
 F 1 "CONN_01X04" V 4799 2062 50  0000 R CNN
-F 2 "" H 4925 2300 50  0001 C CNN
+F 2 "Socket_Strips:Socket_Strip_Straight_1x04" H 4925 2300 50  0001 C CNN
 F 3 "" H 4925 2300 50  0001 C CNN
 	1    4925 2300
@@
 F 0 "P2" V 5915 2062 50  0000 R CNN
 F 1 "CONN_01X04" V 5824 2062 50  0000 R CNN
-F 2 "" H 5950 2300 50  0001 C CNN
+F 2 "Socket_Strips:Socket_Strip_Straight_1x04" H 5950 2300 50  0001 C CNN
 F 3 "" H 5950 2300 50  0001 C CNN
 	1    5950 2300
@@
 F 0 "C1" H 3165 3221 50  0000 L CNN
 F 1 "C" H 3165 3130 50  0000 L CNN
-F 2 "" H 3088 3025 50  0001 C CNN
+F 2 "Capacitors_SMD:C_0805_HandSoldering" H 3088 3025 50  0001 C CNN
 F 3 "" H 3050 3175 50  0001 C CNN
 	1    3050 3175
@@
 F 0 "P3" V 3772 4378 50  0000 L CNN
 F 1 "CONN_01X06" V 3863 4378 50  0000 L CNN
-F 2 "" H 3900 4050 50  0001 C CNN
+F 2 "Socket_Strips:Socket_Strip_Straight_1x06" H 3900 4050 50  0001 C CNN
 F 3 "" H 3900 4050 50  0001 C CNN
 	1    3900 4050
