File: kicad/attiny13aRstbutton/attiny13a.sch (KiCad schematic (older format))
At the start: 7 parts, among them P1 CONN_01X04, P2 CONN_01X04, P3 CONN_01X06, SW1 SWITCH, U1 ATTINY13A-SSU

Commit message: Add capacitor across switch
Parts:
- added C2: C, Capacitors_SMD:C_0805_HandSoldering, symbol C
Connections:
- net rst: now also C2.2
- net at R1.2, SW1.1: now also C2.1
Changed lines of the file:
@@
 rst
 $Comp
-L VCC #PWR01
+L VCC #PWR4
 U 1 1 588CF800
 P 4775 2600
-F 0 "#PWR01" H 4775 2450 50  0001 C CNN
+F 0 "#PWR4" H 4775 2450 50  0001 C CNN
 F 1 "VCC" H 4793 2773 50  0000 C CNN
 F 2 "" H 4775 2600 50  0001 C CNN
@@
 $EndComp
 $Comp
-L GND #PWR02
+L GND #PWR5
 U 1 1 588CF81A
 P 6100 2600
-F 0 "#PWR02" H 6100 2350 50  0001 C CNN
+F 0 "#PWR5" H 6100 2350 50  0001 C CNN
 F 1 "GND" H 6105 2427 50  0000 C CNN
 F 2 "" H 6100 2600 50  0001 C CNN
@@
 $EndComp
 $Comp
-L VCC #PWR03
+L VCC #PWR1
 U 1 1 588CF8A4
 P 1900 3025
-F 0 "#PWR03" H 1900 2875 50  0001 C CNN
+F 0 "#PWR1" H 1900 2875 50  0001 C CNN
 F 1 "VCC" H 1917 3198 50  0000 C CNN
 F 2 "" H 1900 3025 50  0001 C CNN
@@
 $EndComp
 $Comp
-L GND #PWR04
+L GND #PWR2
 U 1 1 588CF8BB
 P 1900 3525
-F 0 "#PWR04" H 1900 3275 50  0001 C CNN
+F 0 "#PWR2" H 1900 3275 50  0001 C CNN
 F 1 "GND" H 1905 3352 50  0000 C CNN
 F 2 "" H 1900 3525 50  0001 C CNN
@@
 $EndComp
 $Comp
-L PWR_FLAG #FLG05
+L PWR_FLAG #FLG1
 U 1 1 588CFAC5
 P 4575 2550
-F 0 "#FLG05" H 4575 2625 50  0001 C CNN
+F 0 "#FLG1" H 4575 2625 50  0001 C CNN
 F 1 "PWR_FLAG" V 4575 2678 50  0000 L CNN
 F 2 "" H 4575 2550 50  0001 C CNN
@@
 $EndComp
 $Comp
-L PWR_FLAG #FLG06
+L PWR_FLAG #FLG2
 U 1 1 588CFAF8
 P 5975 2575
-F 0 "#FLG06" H 5975 2650 50  0001 C CNN
+F 0 "#FLG2" H 5975 2650 50  0001 C CNN
 F 1 "PWR_FLAG" V 5975 2703 50  0000 L CNN
 F 2 "" H 5975 2575 50  0001 C CNN
@@
 $EndComp
 $Comp
-L VCC #PWR07
+L VCC #PWR6
 U 1 1 588CFF9B
 P 6550 2950
-F 0 "#PWR07" H 6550 2800 50  0001 C CNN
+F 0 "#PWR6" H 6550 2800 50  0001 C CNN
 F 1 "VCC" H 6567 3123 50  0000 C CNN
 F 2 "" H 6550 2950 50  0001 C CNN
@@
 $EndComp
 $Comp
-L GND #PWR08
+L GND #PWR7
 U 1 1 588CFFBA
 P 6550 3450
-F 0 "#PWR08" H 6550 3200 50  0001 C CNN
+F 0 "#PWR7" H 6550 3200 50  0001 C CNN
 F 1 "GND" H 6555 3277 50  0000 C CNN
 F 2 "" H 6550 3450 50  0001 C CNN
@@
 Connection ~ 3850 3450
 $Comp
-L GND #PWR09
+L GND #PWR3
 U 1 1 588DE2C4
 P 2350 3450
-F 0 "#PWR09" H 2350 3200 50  0001 C CNN
+F 0 "#PWR3" H 2350 3200 50  0001 C CNN
 F 1 "GND" H 2355 3277 50  0000 C CNN
 F 2 "" H 2350 3450 50  0001 C CNN
@@
 Wire Wire Line
 	2850 3450 2975 3450
+$Comp
+L C C2
+U 1 1 588E01B6
+P 3150 3700
+F 0 "C2" V 3275 3700 50  0000 C CNN
+F 1 "C" V 3025 3700 50  0000 C CNN
+F 2 "Capacitors_SMD:C_0805_HandSoldering" H 3188 3550 50  0001 C CNN
+F 3 "" H 3150 3700 50  0001 C CNN
+	1    3150 3700
+	0    -1   -1   0
+$EndComp
+Wire Wire Line
+	3000 3700 2925 3700
+Wire Wire Line
+	2925 3700 2925 3450
+Connection ~ 2925 3450
+Wire Wire Line
+	3300 3700 3550 3700
+Wire Wire Line
+	3550 3700 3550 3450
+Connection ~ 3550 3450
 $EndSCHEMATC

Commit message: Add 6mm switch button
Parts:
- SW1: footprint Buttons_Switches_ThroughHole:SW_PUSH_SMALL -> Buttons_Switches_ThroughHole:SW_PUSH_6mm
Changed lines of the file:
@@
 F 0 "SW1" H 3175 3687 60  0000 C CNN
 F 1 "SWITCH" H 3175 3581 60  0000 C CNN
-F 2 "Buttons_Switches_ThroughHole:SW_PUSH_SMALL" H 3175 3450 60  0001 C CNN
+F 2 "Buttons_Switches_ThroughHole:SW_PUSH_6mm" H 3175 3450 60  0001 C CNN
 F 3 "" H 3175 3450 60  0000 C CNN
 	1    3175 3450
