File: kicad/attiny13aRstbutton/attiny13a.kicad_pcb (KiCad board)
At the start: 2 copper layers, 28.3 x 21.3 mm, 9 parts, among them P1 CONN_01X04, P2 CONN_01X04, P3 CONN_01X06, SW1 SWITCH, U1 ATTINY13A-SSU

Commit message: Add production ready code
Parts:
- added REF**: M2.2mm, Mounting_Holes:MountingHole_2.2mm_M2, F.Cu at (140.3, 102.6)
Other:
- board size 28.3 x 21.3 mm -> 28.3 x 22.4 mm
Changed lines of the file:
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@@
-(kicad_pcb (version 20160815) (host pcbnew "(2017-01-24 revision 0b6147e)-makepkg")
+(kicad_pcb (version 20170123) (host pcbnew no-vcs-found-7545~57~ubuntu16.04.1)
   (general
     (links 23)
     (no_connects 0)
-    (area 119.558999 83.4245 148.6125 105.5285)
+    (area 119.558999 83.490999 148.030001 105.993001)
     (thickness 1.6)
-    (drawings 25)
+    (drawings 27)
     (tracks 55)
     (zones 0)
-    (modules 9)
+    (modules 10)
     (nets 10)
   )
@@
     (mod_text_size 1 1)
     (mod_text_width 0.15)
-    (pad_size 1.524 1.524)
-    (pad_drill 0.762)
+    (pad_size 2.2 2.2)
+    (pad_drill 2.2)
     (pad_to_mask_clearance 0.2)
     (aux_axis_origin 0 0)
@@
     (tags "SOIC 1.27")
     (attr smd)
-    (fp_text reference U1 (at 0 -3.5) (layer F.SilkS) hide
-      (effects (font (size 1 1) (thickness 0.15)))
+    (fp_text reference U1 (at 0 -3.5) (layer F.SilkS)
+      (effects (font (size 1 1) (thickness 0.15)) hide)
     )
     (fp_text value ATTINY13A-SSU (at -3.844143 0.0855 90) (layer F.SilkS)
@@
     (tags "capacitor 0805")
     (attr smd)
-    (fp_text reference C1 (at -3.556 0 180) (layer F.SilkS) hide
-      (effects (font (size 1 1) (thickness 0.15)))
-    )
-    (fp_text value C (at 0 2.1 180) (layer F.Fab) hide
-      (effects (font (size 1 1) (thickness 0.15)))
+    (fp_text reference C1 (at -3.556 0 180) (layer F.SilkS)
+      (effects (font (size 1 1) (thickness 0.15)) hide)
+    )
+    (fp_text value C (at 0 2.1 180) (layer F.Fab)
+      (effects (font (size 1 1) (thickness 0.15)) hide)
     )
     (fp_line (start -0.5 0.85) (end 0.5 0.85) (layer F.SilkS) (width 0.12))
@@
     (descr "Through hole socket strip")
     (tags "socket strip")
-    (fp_text reference P1 (at -4.572 -6.604 180) (layer F.SilkS) hide
-      (effects (font (size 1 1) (thickness 0.15)))
-    )
-    (fp_text value CONN_01X04 (at -1.905 2.413) (layer F.Fab) hide
-      (effects (font (size 1 1) (thickness 0.15)))
+    (fp_text reference P1 (at -4.572 -6.604 180) (layer F.SilkS)
+      (effects (font (size 1 1) (thickness 0.15)) hide)
+    )
+    (fp_text value CONN_01X04 (at -1.905 2.413) (layer F.Fab)
+      (effects (font (size 1 1) (thickness 0.15)) hide)
     )
     (fp_line (start -1.55 -1.55) (end -1.55 1.55) (layer F.SilkS) (width 0.15))
@@
     (descr "Through hole socket strip")
     (tags "socket strip")
-    (fp_text reference P2 (at 0 -5.1 270) (layer F.SilkS) hide
-      (effects (font (size 1 1) (thickness 0.15)))
-    )
-    (fp_text value CONN_01X04 (at -3.048 -2.667) (layer F.Fab) hide
-      (effects (font (size 1 1) (thickness 0.15)))
+    (fp_text reference P2 (at 0 -5.1 270) (layer F.SilkS)
+      (effects (font (size 1 1) (thickness 0.15)) hide)
+    )
+    (fp_text value CONN_01X04 (at -3.048 -2.667) (layer F.Fab)
+      (effects (font (size 1 1) (thickness 0.15)) hide)
     )
     (fp_line (start -1.75 -1.75) (end -1.75 1.75) (layer F.CrtYd) (width 0.05))
@@
     (descr "Through hole socket strip")
     (tags "socket strip")
-    (fp_text reference P3 (at 0 -6.604 180) (layer F.SilkS) hide
-      (effects (font (size 1 1) (thickness 0.15)))
-    )
-    (fp_text value CONN_01X06 (at 4.445 2.032 90) (layer F.Fab) hide
-      (effects (font (size 1 1) (thickness 0.15)))
+    (fp_text reference P3 (at 0 -6.604 180) (layer F.SilkS)
+      (effects (font (size 1 1) (thickness 0.15)) hide)
+    )
+    (fp_text value CONN_01X06 (at 4.445 2.032 90) (layer F.Fab)
+      (effects (font (size 1 1) (thickness 0.15)) hide)
     )
     (fp_line (start -1.55 -1.55) (end -1.55 1.55) (layer F.SilkS) (width 0.15))
@@
   (module led2layer:superme (layer B.Cu)
     (at 130.937 92.329 180)
-    (fp_text reference G*** (at 0 0 180) (layer B.SilkS) hide
-      (effects (font (thickness 0.3)) (justify mirror))
+    (fp_text reference G*** (at 0 0 180) (layer B.SilkS)
+      (effects (font (thickness 0.3)) (justify mirror) hide)
     )
     (fp_text value "made by ami 2017" (at -5.3975 -1.651 270) (layer B.SilkS)
@@
     (tags "resistor 0805")
     (attr smd)
-    (fp_text reference R1 (at 2.794 0 180) (layer F.SilkS) hide
-      (effects (font (size 1 1) (thickness 0.15)))
+    (fp_text reference R1 (at 2.794 0 180) (layer F.SilkS)
+      (effects (font (size 1 1) (thickness 0.15)) hide)
     )
     (fp_text value 10k (at 0 -1.651 90) (layer F.SilkS)
@@
     )
     (fp_text value C (at 0 2.1 270) (layer F.Fab)
-      (effects (font (size 1 1) (thickness 0.15)))
+      (effects (font (size 1 1) (thickness 0.15)) hide)
     )
     (fp_line (start -0.5 0.85) (end 0.5 0.85) (layer F.SilkS) (width 0.12))
@@
     )
   )
-  (gr_text v0.1 (at 141.224 103.124) (layer F.SilkS)
-    (effects (font (size 1.5 1.5) (thickness 0.3)))
+  (module Mounting_Holes:MountingHole_2.2mm_M2 (layer F.Cu)
+    (at 140.335 102.616)
+    (descr "Mounting Hole 2.2mm, no annular, M2")
+    (tags "mounting hole 2.2mm no annular m2")
+    (fp_text reference REF** (at 0 -3.2) (layer F.SilkS)
+      (effects (font (size 1 1) (thickness 0.15)) hide)
+    )
+    (fp_text value M2.2mm (at -2.286 -0.508 90) (layer F.Fab)
+      (effects (font (size 1 1) (thickness 0.15)) hide)
+    )
+    (fp_circle (center 0 0) (end 2.45 0) (layer F.CrtYd) (width 0.05))
+    (fp_circle (center 0 0) (end 2.2 0) (layer Cmts.User) (width 0.15))
+    (pad "" np_thru_hole circle (at 0 0) (size 2.2 2.2) (drill 2.2) (layers *.Cu *.Mask))
+  )
+  (gr_line (start 147.955 105.918) (end 147.955 104.902) (angle 90) (layer Edge.Cuts) (width 0.15))
+  (gr_line (start 119.634 105.918) (end 147.955 105.918) (angle 90) (layer Edge.Cuts) (width 0.15))
+  (gr_line (start 119.634 104.902) (end 119.634 105.918) (angle 90) (layer Edge.Cuts) (width 0.15))
+  (gr_text v0.1 (at 145.669 102.997 90) (layer F.SilkS)
+    (effects (font (size 1 1) (thickness 0.2)))
   )
   (gr_line (start 147.955 83.566) (end 147.828 83.566) (angle 90) (layer Edge.Cuts) (width 0.15))
   (gr_line (start 147.955 104.902) (end 147.955 83.566) (angle 90) (layer Edge.Cuts) (width 0.15))
-  (gr_line (start 119.634 104.902) (end 147.955 104.902) (angle 90) (layer Edge.Cuts) (width 0.15))
   (gr_line (start 119.634 101.346) (end 119.634 104.902) (angle 90) (layer Edge.Cuts) (width 0.15))
   (gr_text "t13/85 breakout board" (at 131.699 85.0265) (layer F.SilkS)
@@
     (polygon
       (pts
-        (xy 147.32 104.394) (xy 120.142 104.394) (xy 120.142 84.074) (xy 147.32 84.074)
+        (xy 147.32 105.156) (xy 120.142 105.283) (xy 120.142 84.074) (xy 147.32 84.074)
       )
     )
@@
     (polygon
       (pts
-        (xy 147.32 104.394) (xy 120.142 104.394) (xy 120.142 84.074) (xy 147.32 84.074)
+        (xy 147.32 105.156) (xy 120.142 105.283) (xy 120.142 84.074) (xy 147.32 84.074)
       )
     )
