File: kicad/led/panelized.kicad_pcb (KiCad board)
At the start: 2 copper layers, 81.1 x 78.1 mm, 16 parts

Commit message: make it better.
Parts:
- removed the BT1 at (171.8, 89.1)
- removed the BT1 at (171.8, 129.1)
- removed the D1 at (174.4, 74.4)
- removed the D1 at (174.4, 114.4)
- removed the R1 at (192.9, 74.9)
- removed the R1 at (192.9, 114.9)
- removed the REF** at (197.9, 101.6)
- removed the REF** at (197.9, 141.6)
- added BT1: Battery, Battery_Holders:Keystone_103_1x20mm-CoinCell, F.Cu at (168.8, 89.1)
- added BT1: Battery, Battery_Holders:Keystone_103_1x20mm-CoinCell, F.Cu at (168.8, 129.1)
- added D1: LED, LEDs:LED-3MM, F.Cu at (171.4, 74.4)
- added D1: LED, LEDs:LED-3MM, F.Cu at (171.4, 114.4)
- added R1: 100, Resistors_SMD:R_0603_HandSoldering, F.Cu at (189.9, 74.9)
- added R1: 100, Resistors_SMD:R_0603_HandSoldering, F.Cu at (189.9, 114.9)
- added REF**: 1pin, Connectors:1pin, F.Cu at (194.9, 101.6)
- added REF**: 1pin, Connectors:1pin, F.Cu at (194.9, 141.6)
Other:
- board size 81.1 x 78.1 mm -> 78.1 x 78.1 mm
Changed lines of the file:
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@@
   )
   (module Battery_Holders:Keystone_103_1x20mm-CoinCell (layer F.Cu)
-    (at 171.790001 89.075074 0)
+    (at 168.790001 89.075074 0)
     (descr http://www.keyelco.com/product-pdf.cfm?p=719)
     (tags "Keystone type 103 battery holder")
@@
   )
   (module LEDs:LED-3MM (layer F.Cu)
-    (at 174.44 74.375 180)
+    (at 171.44 74.375 180)
     (descr "LED 3mm round vertical")
     (tags "LED  3mm round vertical")
@@
   )
   (module Resistors_SMD:R_0603_HandSoldering (layer F.Cu)
-    (at 192.86 74.93 90)
+    (at 189.86 74.93 90)
     (descr "Resistor SMD 0603, hand soldering")
     (tags "resistor 0603")
@@
   )
   (module Connectors:1pin (layer F.Cu)
-    (at 197.94 101.6 0)
+    (at 194.94 101.6 0)
     (descr "module 1 pin (ou trou mecanique de percage)")
     (tags DEV)
@@
   )
   (module Battery_Holders:Keystone_103_1x20mm-CoinCell (layer F.Cu)
-    (at 171.790001 129.075074 0)
+    (at 168.790001 129.075074 0)
     (descr http://www.keyelco.com/product-pdf.cfm?p=719)
     (tags "Keystone type 103 battery holder")
@@
   )
   (module LEDs:LED-3MM (layer F.Cu)
-    (at 174.44 114.375 180)
+    (at 171.44 114.375 180)
     (descr "LED 3mm round vertical")
     (tags "LED  3mm round vertical")
@@
   )
   (module Resistors_SMD:R_0603_HandSoldering (layer F.Cu)
-    (at 192.86 114.93 90)
+    (at 189.86 114.93 90)
     (descr "Resistor SMD 0603, hand soldering")
     (tags "resistor 0603")
@@
   )
   (module Connectors:1pin (layer F.Cu)
-    (at 197.94 141.6 0)
+    (at 194.94 141.6 0)
     (descr "module 1 pin (ou trou mecanique de percage)")
     (tags DEV)
@@
   (gr_line (start 121.92 106.68) (end 160.02 106.68) (angle 90) (layer Edge.Cuts) (width 0.15))
   (gr_line (start 121.92 68.58) (end 121.92 106.68) (angle 90) (layer Edge.Cuts) (width 0.15))
-  (gr_text "LED Board v0.1" (at 177.62 101.6 0) (layer B.Cu)
+  (gr_text "LED Board v0.1" (at 174.62 101.6 0) (layer B.Cu)
     (effects (font (size 1.5 1.5) (thickness 0.3)) (justify mirror))
   )
-  (gr_line (start 203.02 68.58) (end 164.92 68.58) (angle 90) (layer Edge.Cuts) (width 0.15))
-  (gr_line (start 203.02 106.68) (end 203.02 68.58) (angle 90) (layer Edge.Cuts) (width 0.15))
-  (gr_line (start 164.92 106.68) (end 203.02 106.68) (angle 90) (layer Edge.Cuts) (width 0.15))
-  (gr_line (start 164.92 68.58) (end 164.92 106.68) (angle 90) (layer Edge.Cuts) (width 0.15))
-  (gr_text "LED Board v0.1" (at 177.62 141.6 0) (layer B.Cu)
+  (gr_line (start 200.02 68.58) (end 161.92 68.58) (angle 90) (layer Edge.Cuts) (width 0.15))
+  (gr_line (start 200.02 106.68) (end 200.02 68.58) (angle 90) (layer Edge.Cuts) (width 0.15))
+  (gr_line (start 161.92 106.68) (end 200.02 106.68) (angle 90) (layer Edge.Cuts) (width 0.15))
+  (gr_line (start 161.92 68.58) (end 161.92 106.68) (angle 90) (layer Edge.Cuts) (width 0.15))
+  (gr_text "LED Board v0.1" (at 174.62 141.6 0) (layer B.Cu)
     (effects (font (size 1.5 1.5) (thickness 0.3)) (justify mirror))
   )
-  (gr_line (start 203.02 108.58) (end 164.92 108.58) (angle 90) (layer Edge.Cuts) (width 0.15))
-  (gr_line (start 203.02 146.68) (end 203.02 108.58) (angle 90) (layer Edge.Cuts) (width 0.15))
-  (gr_line (start 164.92 146.68) (end 203.02 146.68) (angle 90) (layer Edge.Cuts) (width 0.15))
-  (gr_line (start 164.92 108.58) (end 164.92 146.68) (angle 90) (layer Edge.Cuts) (width 0.15))
+  (gr_line (start 200.02 108.58) (end 161.92 108.58) (angle 90) (layer Edge.Cuts) (width 0.15))
+  (gr_line (start 200.02 146.68) (end 200.02 108.58) (angle 90) (layer Edge.Cuts) (width 0.15))
+  (gr_line (start 161.92 146.68) (end 200.02 146.68) (angle 90) (layer Edge.Cuts) (width 0.15))
+  (gr_line (start 161.92 108.58) (end 161.92 146.68) (angle 90) (layer Edge.Cuts) (width 0.15))
   (gr_text "LED Board v0.1" (at 134.62 141.6 0) (layer B.Cu)
     (effects (font (size 1.5 1.5) (thickness 0.3)) (justify mirror))
@@
   (segment (start 131.44 74.375) (end 130.81 74.93) (width 0.25) (layer B.Cu) (net 3) (status 80000))
   (segment (start 131.44 74.375) (end 130.81 74.93) (width 0.25) (layer B.Cu) (net 3) (status 80000))
-  (segment (start 171.790001 89.075074) (end 171.27 88.9) (width 0.25) (layer F.Cu) (net 5))
-  (segment (start 171.27 88.9) (end 171.27 74.93) (width 0.25) (layer F.Cu) (net 5))
-  (segment (start 171.27 74.93) (end 171.9 74.375) (width 0.25) (layer F.Cu) (net 5))
-  (segment (start 171.27 88.9) (end 171.790001 89.075074) (width 0.25) (layer F.Cu) (net 5))
-  (segment (start 171.9 74.375) (end 171.27 74.93) (width 0.25) (layer F.Cu) (net 5))
-  (segment (start 192.86 73.83) (end 174.985 73.83) (width 0.25) (layer F.Cu) (net 6))
-  (segment (start 174.985 73.83) (end 174.44 74.375) (width 0.25) (layer F.Cu) (net 6))
-  (segment (start 192.86 73.66) (end 192.86 73.83) (width 0.25) (layer F.Cu) (net 6))
-  (segment (start 192.86 73.66) (end 192.86 73.83) (width 0.25) (layer F.Cu) (net 6))
-  (segment (start 174.44 74.375) (end 173.81 74.93) (width 0.25) (layer B.Cu) (net 6))
-  (segment (start 174.44 74.375) (end 173.81 74.93) (width 0.25) (layer B.Cu) (net 6))
-  (segment (start 171.790001 129.075074) (end 171.27 128.9) (width 0.25) (layer F.Cu) (net 8))
-  (segment (start 171.27 128.9) (end 171.27 114.93) (width 0.25) (layer F.Cu) (net 8))
-  (segment (start 171.27 114.93) (end 171.9 114.375) (width 0.25) (layer F.Cu) (net 8))
-  (segment (start 171.27 128.9) (end 171.790001 129.075074) (width 0.25) (layer F.Cu) (net 8))
-  (segment (start 171.9 114.375) (end 171.27 114.93) (width 0.25) (layer F.Cu) (net 8))
-  (segment (start 192.86 113.83) (end 174.985 113.83) (width 0.25) (layer F.Cu) (net 9))
-  (segment (start 174.985 113.83) (end 174.44 114.375) (width 0.25) (layer F.Cu) (net 9))
-  (segment (start 192.86 113.66) (end 192.86 113.83) (width 0.25) (layer F.Cu) (net 9))
-  (segment (start 192.86 113.66) (end 192.86 113.83) (width 0.25) (layer F.Cu) (net 9))
-  (segment (start 174.44 114.375) (end 173.81 114.93) (width 0.25) (layer B.Cu) (net 9))
-  (segment (start 174.44 114.375) (end 173.81 114.93) (width 0.25) (layer B.Cu) (net 9))
+  (segment (start 168.790001 89.075074) (end 168.27 88.9) (width 0.25) (layer F.Cu) (net 5))
+  (segment (start 168.27 88.9) (end 168.27 74.93) (width 0.25) (layer F.Cu) (net 5))
+  (segment (start 168.27 74.93) (end 168.9 74.375) (width 0.25) (layer F.Cu) (net 5))
+  (segment (start 168.27 88.9) (end 168.790001 89.075074) (width 0.25) (layer F.Cu) (net 5))
+  (segment (start 168.9 74.375) (end 168.27 74.93) (width 0.25) (layer F.Cu) (net 5))
+  (segment (start 189.86 73.83) (end 171.985 73.83) (width 0.25) (layer F.Cu) (net 6))
+  (segment (start 171.985 73.83) (end 171.44 74.375) (width 0.25) (layer F.Cu) (net 6))
+  (segment (start 189.86 73.66) (end 189.86 73.83) (width 0.25) (layer F.Cu) (net 6))
+  (segment (start 189.86 73.66) (end 189.86 73.83) (width 0.25) (layer F.Cu) (net 6))
+  (segment (start 171.44 74.375) (end 170.81 74.93) (width 0.25) (layer B.Cu) (net 6))
+  (segment (start 171.44 74.375) (end 170.81 74.93) (width 0.25) (layer B.Cu) (net 6))
+  (segment (start 168.790001 129.075074) (end 168.27 128.9) (width 0.25) (layer F.Cu) (net 8))
+  (segment (start 168.27 128.9) (end 168.27 114.93) (width 0.25) (layer F.Cu) (net 8))
+  (segment (start 168.27 114.93) (end 168.9 114.375) (width 0.25) (layer F.Cu) (net 8))
+  (segment (start 168.27 128.9) (end 168.790001 129.075074) (width 0.25) (layer F.Cu) (net 8))
+  (segment (start 168.9 114.375) (end 168.27 114.93) (width 0.25) (layer F.Cu) (net 8))
+  (segment (start 189.86 113.83) (end 171.985 113.83) (width 0.25) (layer F.Cu) (net 9))
+  (segment (start 171.985 113.83) (end 171.44 114.375) (width 0.25) (layer F.Cu) (net 9))
+  (segment (start 189.86 113.66) (end 189.86 113.83) (width 0.25) (layer F.Cu) (net 9))
+  (segment (start 189.86 113.66) (end 189.86 113.83) (width 0.25) (layer F.Cu) (net 9))
+  (segment (start 171.44 114.375) (end 170.81 114.93) (width 0.25) (layer B.Cu) (net 9))
+  (segment (start 171.44 114.375) (end 170.81 114.93) (width 0.25) (layer B.Cu) (net 9))
   (segment (start 128.790001 129.075074) (end 128.27 128.9) (width 0.25) (layer F.Cu) (net 11))
   (segment (start 128.27 128.9) (end 128.27 114.93) (width 0.25) (layer F.Cu) (net 11))
@@
     (polygon
       (pts
-        (xy 200.48 104.14) (xy 167.46 104.14) (xy 167.46 69.85) (xy 200.48 69.85)
+        (xy 197.48 104.14) (xy 164.46 104.14) (xy 164.46 69.85) (xy 197.48 69.85)
       )
     )
@@
     (polygon
       (pts
-        (xy 200.48 144.14) (xy 167.46 144.14) (xy 167.46 109.85) (xy 200.48 109.85)
+        (xy 197.48 144.14) (xy 164.46 144.14) (xy 164.46 109.85) (xy 197.48 109.85)
       )
     )
