File: kicad/breadboard/esp12e.sch (KiCad schematic (older format))
At the start: 9 parts, among them J1 Conn_01x08, J3 Conn_01x08, SW1 SWITCH, SW2 SWITCH, U3 ESP-12E

Commit message: fix sch
Changed lines of the file:
@@
 $Descr A4 11693 8268
 encoding utf-8
-Sheet 3 4
+Sheet 3 3
 Title ""
 Date ""
@@
 	7700 2975 6900 2975
 Connection ~ 6900 2975
-Text GLabel 4850 3825 0    60   Input ~ 0
-V3.3v
-$Comp
-L GND #PWR014
+$Comp
+L GND #PWR013
 U 1 1 5A086174
 P 5250 4525
-F 0 "#PWR014" H 5250 4275 50  0001 C CNN
+F 0 "#PWR013" H 5250 4275 50  0001 C CNN
 F 1 "GND" H 5250 4375 50  0000 C CNN
 F 2 "" H 5250 4525 50  0001 C CNN
@@
 $EndComp
 $Comp
-L GND #PWR015
+L GND #PWR014
 U 1 1 5A08618F
 P 6850 4525
-F 0 "#PWR015" H 6850 4275 50  0001 C CNN
+F 0 "#PWR014" H 6850 4275 50  0001 C CNN
 F 1 "GND" H 6850 4375 50  0000 C CNN
 F 2 "" H 6850 4525 50  0001 C CNN
@@
 	6900 3975 6900 3825
 $Comp
-L GND #PWR016
+L GND #PWR015
 U 1 1 5A086160
 P 6900 3975
-F 0 "#PWR016" H 6900 3725 50  0001 C CNN
+F 0 "#PWR015" H 6900 3725 50  0001 C CNN
 F 1 "GND" H 6900 3825 50  0000 C CNN
 F 2 "" H 6900 3975 50  0001 C CNN
@@
 NoConn ~ 5950 4325
 NoConn ~ 6050 4325
-Text GLabel 4950 4850 0    60   Input ~ 0
-GND
-$Comp
-L GND #PWR017
-U 1 1 5A090755
-P 4950 4850
-F 0 "#PWR017" H 4950 4600 50  0001 C CNN
-F 1 "GND" H 4950 4700 50  0000 C CNN
-F 2 "" H 4950 4850 50  0001 C CNN
-F 3 "" H 4950 4850 50  0001 C CNN
-	1    4950 4850
-	0    -1   -1   0
-$EndComp
+Text GLabel 4275 4150 0    60   Input ~ 0
+V3.3v
+Wire Wire Line
+	4275 4150 4350 4150
+Wire Wire Line
+	4350 4150 4350 4025
+Wire Wire Line
+	4350 4025 4900 4025
+Wire Wire Line
+	4900 4025 4900 3825
 $EndSCHEMATC
