File: projects/kicad6/esp01-programming-board/esp01-programming/esp01-programming.kicad_sch (KiCad schematic)
At the start: 20 parts, among them J1 Conn_01x06_Female, J2 Conn_01x05_Female, SW1 SW_DIP_x01, SW2 SW_DIP_x01, U1 AMS1117-3.3, U2 ESP01

Commit message: Add new changes
Parts:
- removed C2: 2.2u, Capacitor_THT:C_Radial_D4.0mm_H7.0mm_P1.50mm, symbol Device:C_Polarized
- removed C3: 220u, Capacitor_THT:C_Radial_D4.0mm_H7.0mm_P1.50mm, symbol Device:C
- removed D1: D, Diode_SMD:D_1206_3216Metric_Pad1.42x1.75mm_HandSolder, symbol Device:D
- removed J2: Conn_01x05_Female, Connector_PinHeader_2.54mm:PinHeader_1x05_P2.54mm_Vertical, symbol Connector:Conn_01x05_Female
- added C2: 47u, Capacitor_SMD:C_0805_2012Metric_Pad1.18x1.45mm_HandSolder, symbol Device:C
- added J3: RTS pinout, MY_ETCHING:PinSocket_1x02_P2.54mm_Vertical_ETCH, symbol Connector:Conn_01x02_Female
- added Q1, Q2, Q3, Q4: 2N3904, Package_TO_SOT_THT:TO-92_Wide, symbol Transistor_BJT:2N3904
- added R10, R11, R12, R7, R8, R9: 10k, Resistor_SMD:R_0805_2012Metric_Pad1.20x1.40mm_HandSolder, symbol Device:R
- C1: value 100u -> 10u; footprint Capacitor_THT:C_Radial_D4.0mm_H7.0mm_P1.50mm -> Capacitor_SMD:C_0805_2012Metric_Pad1.18x1.45mm_HandSolder
- J1: value Conn_01x06_Female -> FT232RL header
- R1: value 680 -> 10k
Connections:
- net +5V: now also J1.4 (Pin_4), R12.1, R9.1
- net 3.3v: now also C2.1, R10.1, R11.1, R7.2, R8.2; no longer R2.1
- net DTR: now also Q2.1 (E)
- net GND: now also C2.2; no longer R1.2
- net PRG: now also Q2.3 (C)
- net uC_RST: now also Q1.3 (C); no longer R2.2
- net uC_RX: now also Q3.1 (E), R7.1; no longer R4.1
- net uC_TX: now also Q4.1 (E), R10.2; no longer R3.2
- new net: Q3.2 (B), R8.1
- new net: Q4.2 (B), R11.2
- new net: Q2.2 (B), R2.2
- new net: Q1.2 (B), R1.2
- new net RTS: J3.1 (Pin_1), J3.2 (Pin_2), Q1.1 (E), R2.1
- new net ft_RX: Q4.3 (C), R12.2, R3.2
- new net ft_TX: Q3.3 (C), R4.1, R9.2
- no-connect marks 5 -> 1
Other:
- moved on the sheet: J1, R3, R4
