File: projects/kicad6/esp01-porch-lightv2/esp01-porch-lightv2.kicad_pcb (KiCad board)
At the start: 2 copper layers, 49.3 x 40.9 mm, 15 parts, among them J1 Relay, J2 Power_IN, Q1 2N3904, U1 AMS1117-3.3, U2 ESP01

Commit message: esp porch ligh v2: finished
Parts:
- removed C4: 470u, Capacitor_THT:C_Radial_D4.0mm_H7.0mm_P1.50mm
- removed R4, R5: 10k, Resistor_SMD:R_0805_2012Metric_Pad1.20x1.40mm_HandSolder
- added Q2: 2N3906, Package_TO_SOT_THT:TO-92_Wide, F.Cu at (92.2, 131.9)
- J2: value Power_IN -> Conn_01x02_Male
- R2: value 10k -> 1k
- moved R3 26.9 mm to (97.0, 121.2)
- moved R2 24.4 mm to (96.2, 137.9), turned to 0 degrees
- moved Q1 14.6 mm to (101.3, 131.8)
- moved R6 14.6 mm to (104.6, 122.6)
- moved J1 14.6 mm to (109.6, 124.4)
- moved R1 1.95 mm to (74.2, 138.5)
Connections:
- R2 pad 2: 3.3v -> Net-(Q2-Pad2)
- R3 pad 1: GPIO2 -> Net-(Q2-Pad3)
Routing:
- net Net-(Q1-Pad2): track 24.9 -> 8.89 mm
- net 3.3v: track 64.8 -> 49.3 mm
- net Net-(Q2-Pad2): track 0.00 -> 14.6 mm
- net RELAY_IN: track 28.6 -> 14.1 mm
- net GPIO2: track 16.6 -> 24.8 mm, vias 0 -> 1
- net Net-(Q2-Pad3): track 0.00 -> 7.22 mm
- net +5V: track 63.0 -> 64.7 mm
Other:
- board size 49.3 x 40.9 mm -> 51.5 x 39.1 mm
