File: projects/kicad6/esp01-porch-lightv2/esp01-porch-lightv2.kicad_sch (KiCad schematic)
At the start: 14 parts, among them J1 Relay, J2 Conn_01x02_Male, Q1 2N3904, Q2 2N3906, U1 AMS1117-3.3, U2 ESP01

Commit message: esp porch ligh v2: finished
Parts:
- removed C4: 470u, Capacitor_THT:C_Radial_D4.0mm_H7.0mm_P1.50mm, symbol Device:C
- Q2: footprint Package_TO_SOT_THT:TO-92_Inline -> Package_TO_SOT_THT:TO-92_Wide
Other:
- moved on the sheet: J1, Q1, R3, R6
