File: projects/led/led.kicad_sch (KiCad schematic)
At the start: 3 parts, among them J1 Conn_01x02_Pin

Commit message: add more
Parts:
- added H1, H2: MountingHole, MountingHole:MountingHole_2.2mm_M2_DIN965, symbol Mechanical:MountingHole
Other:
- note added: "CNC sample project - first"
Changed lines of the file:
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@@
 	(generator_version "9.0")
 	(paper "A4")
+	(rectangle
+		(start 127 41.91)
+		(end 190.5 71.12)
+		(stroke
+			(width 0)
+			(type dash)
+		)
+		(fill
+			(type none)
+		)
+	)
+	(text "CNC sample project - first"
+		(exclude_from_sim no)
+		(at 141.478 45.212 0)
+		(effects
+			(font
+				(size 1.27 1.27)
+			)
+		)
+	)
 	(junction
 		(at 160.02 63.5)
@@
 	(symbol
 		(lib_id "power:PWR_FLAG")
-		(at 123.19 60.96 0)
+		(at 180.34 50.8 0)
 		(unit 1)
 		(exclude_from_sim no)
@@
 		(fields_autoplaced yes)
 		(property "Reference" "#FLG01"
-			(at 123.19 59.055 0)
+			(at 180.34 48.895 0)
 			(effects
 				(font
@@
 		)
 		(property "Value" "PWR_FLAG"
-			(at 123.19 55.88 0)
+			(at 180.34 45.72 0)
 			(effects
 				(font
@@
 		)
 		(property "Footprint" ""
-			(at 123.19 60.96 0)
+			(at 180.34 50.8 0)
 			(effects
 				(font
@@
 		)
 		(property "Datasheet" "~"
-			(at 123.19 60.96 0)
+			(at 180.34 50.8 0)
 			(effects
 				(font
@@
 		)
 		(property "Description" "Special symbol for telling ERC where power comes from"
-			(at 123.19 60.96 0)
+			(at 180.34 50.8 0)
 			(effects
 				(font
@@
 				(path "/c7dc96e4-6e5e-4093-850b-98ec6b01f332"
 					(reference "#FLG01")
+					(unit 1)
+				)
+			)
+		)
+	)
+	(symbol
+		(lib_id "Mechanical:MountingHole")
+		(at 186.69 68.58 0)
+		(unit 1)
+		(exclude_from_sim no)
+		(in_bom no)
+		(on_board yes)
+		(dnp no)
+		(fields_autoplaced yes)
+		(property "Reference" "H2"
+			(at 189.23 67.3099 0)
+			(effects
+				(font
+					(size 1.27 1.27)
+				)
+				(justify left)
+			)
+		)
+		(property "Value" "MountingHole"
+			(at 189.23 69.8499 0)
+			(effects
+				(font
+					(size 1.27 1.27)
+				)
+				(justify left)
+			)
+		)
+		(property "Footprint" "MountingHole:MountingHole_2.2mm_M2_DIN965"
+			(at 186.69 68.58 0)
+			(effects
+				(font
+					(size 1.27 1.27)
+				)
+				(hide yes)
+			)
+		)
+		(property "Datasheet" "~"
+			(at 186.69 68.58 0)
+			(effects
+				(font
+					(size 1.27 1.27)
+				)
+				(hide yes)
+			)
+		)
+		(property "Description" "Mounting Hole without connection"
+			(at 186.69 68.58 0)
+			(effects
+				(font
+					(size 1.27 1.27)
+				)
+				(hide yes)
+			)
+		)
+		(instances
+			(project ""
+				(path "/c7dc96e4-6e5e-4093-850b-98ec6b01f332"
+					(reference "H2")
 					(unit 1)
 				)
@@
 	(symbol
 		(lib_id "power:PWR_FLAG")
-		(at 114.3 60.96 180)
+		(at 171.45 50.8 180)
 		(unit 1)
 		(exclude_from_sim no)
@@
 		(fields_autoplaced yes)
 		(property "Reference" "#FLG02"
-			(at 114.3 62.865 0)
+			(at 171.45 52.705 0)
 			(effects
 				(font
@@
 		)
 		(property "Value" "PWR_FLAG"
-			(at 114.3 66.04 0)
+			(at 171.45 55.88 0)
 			(effects
 				(font
@@
 		)
 		(property "Footprint" ""
-			(at 114.3 60.96 0)
+			(at 171.45 50.8 0)
 			(effects
 				(font
@@
 		)
 		(property "Datasheet" "~"
-			(at 114.3 60.96 0)
+			(at 171.45 50.8 0)
 			(effects
 				(font
@@
 		)
 		(property "Description" "Special symbol for telling ERC where power comes from"
-			(at 114.3 60.96 0)
+			(at 171.45 50.8 0)
 			(effects
 				(font
@@
 	(symbol
 		(lib_id "power:GND")
-		(at 123.19 60.96 0)
+		(at 180.34 50.8 0)
 		(unit 1)
 		(exclude_from_sim no)
@@
 		(fields_autoplaced yes)
 		(property "Reference" "#PWR02"
-			(at 123.19 67.31 0)
+			(at 180.34 57.15 0)
 			(effects
 				(font
@@
 		)
 		(property "Value" "GND"
-			(at 123.19 66.04 0)
+			(at 180.34 55.88 0)
 			(effects
 				(font
@@
 		)
 		(property "Footprint" ""
-			(at 123.19 60.96 0)
+			(at 180.34 50.8 0)
 			(effects
 				(font
@@
 		)
 		(property "Datasheet" ""
-			(at 123.19 60.96 0)
+			(at 180.34 50.8 0)
 			(effects
 				(font
@@
 		)
 		(property "Description" "Power symbol creates a global label with name \"GND\" , ground"
-			(at 123.19 60.96 0)
+			(at 180.34 50.8 0)
 			(effects
 				(font
@@
 	(symbol
 		(lib_id "power:VCC")
-		(at 114.3 60.96 0)
+		(at 171.45 50.8 0)
 		(unit 1)
 		(exclude_from_sim no)
@@
 		(fields_autoplaced yes)
 		(property "Reference" "#PWR01"
-			(at 114.3 64.77 0)
+			(at 171.45 54.61 0)
 			(effects
 				(font
@@
 		)
 		(property "Value" "VCC"
-			(at 114.3 55.88 0)
+			(at 171.45 45.72 0)
 			(effects
 				(font
@@
 		)
 		(property "Footprint" ""
-			(at 114.3 60.96 0)
+			(at 171.45 50.8 0)
 			(effects
 				(font
@@
 		)
 		(property "Datasheet" ""
-			(at 114.3 60.96 0)
+			(at 171.45 50.8 0)
 			(effects
 				(font
@@
 		)
 		(property "Description" "Power symbol creates a global label with name \"VCC\""
-			(at 114.3 60.96 0)
+			(at 171.45 50.8 0)
 			(effects
 				(font
@@
 					(unit 1)
 				)
+			)
+		)
+	)
+	(symbol
+		(lib_id "Mechanical:MountingHole")
+		(at 130.81 67.31 0)
+		(unit 1)
+		(exclude_from_sim no)
+		(in_bom no)
+		(on_board yes)
+		(dnp no)
+		(fields_autoplaced yes)
+		(property "Reference" "H1"
+			(at 133.35 66.0399 0)
+			(effects
+				(font
+					(size 1.27 1.27)
+				)
+				(justify left)
+			)
+		)
+		(property "Value" "MountingHole"
+			(at 133.35 68.5799 0)
+			(effects
+				(font
+					(size 1.27 1.27)
+				)
+				(justify left)
+			)
+		)
+		(property "Footprint" "MountingHole:MountingHole_2.2mm_M2_DIN965"
+			(at 130.81 67.31 0)
+			(effects
+				(font
+					(size 1.27 1.27)
+				)
+				(hide yes)
+			)
+		)
+		(property "Datasheet" "~"
+			(at 130.81 67.31 0)
+			(effects
+				(font
+					(size 1.27 1.27)
+				)
+				(hide yes)
+			)
+		)
+		(property "Description" "Mounting Hole without connection"
+			(at 130.81 67.31 0)
+			(effects
+				(font
+					(size 1.27 1.27)
+				)
+				(hide yes)
+			)
+		)
+		(instances
+			(project ""
+				(path "/c7dc96e4-6e5e-4093-850b-98ec6b01f332"
+					(reference "H1")
+					(unit 1)
+				)
