File: solidcraft/rpi5-fan-case/rpi5-fan-pwm-controller/rpi5-fan-pwm-controller.kicad_sch (KiCad schematic)
At the start: 0 parts

Commit message: fix firmware
Parts:
- added C1: 100uF, symbol Device:C
- added Q1: 2N3904, Package_TO_SOT_THT:TO-92_Inline, symbol Transistor_BJT:2N3904
- added R1: 1k, symbol Device:R
- added R2: 10k, symbol Device:R
- added U1: ESP-01, RF_Module:ESP-01, symbol RF_Module:ESP-01
- added U2: LM2596S-3.3, Package_TO_SOT_SMD:TO-263-5_TabPin3, symbol Regulator_Switching:LM2596S-3.3
Connections:
- new net: C1.2, U1.8 (VCC), U2.2 (OUT)
- new net: Q1.2 (B), R1.1, R2.1
- new net +12V: U2.1 (VIN)
- new net FAN_PWM: Q1.3 (C)
- new net GND: C1.1, Q1.1 (E), R2.2, U1.1 (GND), U2.3 (GND)
- new net PWM: R1.2, U1.5 (TXD/IO1)
Other:
- note added: "ESP01S"
- note added: "LM2596 DC-DC"

Commit message: Add working stuff
Parts:
- added C2: 22pF, symbol Device:C
- R1: value 1k -> 10k
Connections:
- net FAN_PWM: now also U1.5 (TXD/IO1)
- net GND: now also C2.2; no longer R2.2
- net PWM: now also R2.2; no longer U1.5 (TXD/IO1)
- net at C1.2, U1.8 (VCC), U2.2 (OUT): now also C2.1
- net at Q1.2 (B), R1.1: no longer R2.1
- new net +3.3V: R2.1
Other:
- note added: "Without 10k pullup on tx pin, esp01s (blue led) does not boot. It boots with 10k pullup when nothing is connected to tx pin."
